File: board/Electronicsmb.brd (EAGLE design)
At the start: 96 x 70 mm, 17 parts

Commit message: minor tweaks
Connections:
- new net RAW: J1.2, U$1.RAW
- net VCC: no longer J1.2
Routing:
- net RAW: track 0.00 -> 60.8 mm
- net VCC: track 97.9 -> 46.2 mm
- net N$2: track 213.3 -> 189.7 mm
- net D1: track 49.4 -> 67.8 mm
- net GND: track 147.7 -> 155.3 mm, vias 1 -> 0
- net N$27: track 64.3 -> 62.3 mm
- net D2: track 35.8 -> 36.3 mm

Commit message: final tweaks to V1 and starter code
Parts:
- R2: device resistor:0204/7 -> SparkFun:AXIAL-0.4
Connections:
- removed net D1: D1.A, U$1.RX1
- removed net N$1: S1.2, U$1.TX0
- new net A1: D1.A, U$1.A1
- new net A3: S1.2, U$1.A3
- net GND: now also R2.P$2; no longer R2.2
- net N$2: now also R2.P$1; no longer R2.1
Routing:
- net D1: track 67.8 -> 0.00 mm
- net A3: track 0.00 -> 40.1 mm
- net N$1: track 37.4 -> 0.00 mm
- net A1: track 0.00 -> 34.8 mm
- net N$27: track 62.3 -> 64.6 mm
- net GND: track 155.3 -> 153.1 mm, vias 0 -> 1
- net D2: track 36.3 -> 34.3 mm
- net N$2: track 189.7 -> 188.0 mm
- net RAW: track 60.8 -> 59.3 mm
- net D9: track 43.8 -> 44.8 mm
