File: board/Electronicsmb.sch (EAGLE design)
At the start: 17 parts

Commit message: minor tweaks
Connections:
- new net RAW: J1.2, U$1.RAW
- net VCC: no longer J1.2
Changed lines of the file:
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@@
 <part name="P+1" library="supply1" library_urn="urn:adsk.eagle:library:371" deviceset="VCC" device=""/>
 <part name="J1" library="SparkFun-Connectors" library_urn="urn:adsk.eagle:library:513" deviceset="CONN_02" device="" package3d_urn="urn:adsk.eagle:package:38039/1"/>
-<part name="P+3" library="supply1" library_urn="urn:adsk.eagle:library:371" deviceset="VCC" device=""/>
 <part name="SUPPLY3" library="supply2" library_urn="urn:adsk.eagle:library:372" deviceset="GND" device=""/>
 <part name="SUPPLY4" library="supply2" library_urn="urn:adsk.eagle:library:372" deviceset="GND" device=""/>
@@
 <instance part="P+1" gate="VCC" x="50.8" y="68.58" rot="R270"/>
 <instance part="J1" gate="G$1" x="22.86" y="132.08"/>
-<instance part="P+3" gate="VCC" x="35.56" y="134.62" rot="R270"/>
 <instance part="SUPPLY3" gate="GND" x="35.56" y="132.08" rot="R90"/>
 <instance part="SUPPLY4" gate="GND" x="124.46" y="101.6" rot="R90"/>
@@
 <pinref part="P+1" gate="VCC" pin="VCC"/>
 <wire x1="45.72" y1="68.58" x2="48.26" y2="68.58" width="0.1524" layer="91"/>
-</segment>
-<segment>
-<pinref part="J1" gate="G$1" pin="2"/>
-<pinref part="P+3" gate="VCC" pin="VCC"/>
-<wire x1="30.48" y1="134.62" x2="33.02" y2="134.62" width="0.1524" layer="91"/>
 </segment>
 </net>
@@
 </segment>
 </net>
+<net name="RAW" class="0">
+<segment>
+<pinref part="U$1" gate="G$1" pin="RAW"/>
+<wire x1="78.74" y1="93.98" x2="76.2" y2="93.98" width="0.1524" layer="91"/>
+<label x="71.12" y="91.44" size="1.778" layer="95"/>
+</segment>
+<segment>
+<pinref part="J1" gate="G$1" pin="2"/>
+<wire x1="30.48" y1="134.62" x2="33.02" y2="134.62" width="0.1524" layer="91"/>
+<label x="35.56" y="134.62" size="1.778" layer="95"/>
+</segment>
+</net>

Commit message: final tweaks to V1 and starter code
Parts:
- R2: device resistor:R-US_0204/7 -> SparkFun:RESISTORPTH-1/4W
Connections:
- removed net D1: D1.A, U$1.RX1
- removed net N$1: S1.S, U$1.TX0
- new net A1: D1.A, U$1.A1
- new net A3: S1.S, U$1.A3
Other:
- moved on the sheet: S1
Changed lines of the file:
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@@
 <part name="SUPPLY4" library="supply2" library_urn="urn:adsk.eagle:library:372" deviceset="GND" device=""/>
 <part name="SUPPLY6" library="supply2" library_urn="urn:adsk.eagle:library:372" deviceset="GND" device=""/>
-<part name="R2" library="resistor" library_urn="urn:adsk.eagle:library:348" deviceset="R-US_" device="0204/7" package3d_urn="urn:adsk.eagle:package:25945/1" value="270"/>
+<part name="R2" library="SparkFun" deviceset="RESISTOR" device="PTH-1/4W" value="270"/>
 <part name="SUPPLY1" library="supply2" library_urn="urn:adsk.eagle:library:372" deviceset="GND" device=""/>
 </parts>
@@
 <instance part="D11" gate="G$1" x="195.58" y="73.66" rot="R90"/>
 <instance part="D12" gate="G$1" x="195.58" y="66.04" rot="R90"/>
-<instance part="S1" gate="1" x="129.54" y="93.98" rot="R90"/>
+<instance part="S1" gate="1" x="93.98" y="66.04" rot="R90"/>
 <instance part="U$2" gate="G$1" x="48.26" y="66.04" rot="R90"/>
 <instance part="SUPPLY2" gate="GND" x="25.4" y="68.58" rot="R270"/>
@@
 <instance part="SUPPLY6" gate="GND" x="73.66" y="96.52" rot="R270"/>
 <instance part="R2" gate="G$1" x="215.9" y="104.14"/>
-<instance part="SUPPLY1" gate="GND" x="139.7" y="93.98" rot="R90"/>
+<instance part="SUPPLY1" gate="GND" x="104.14" y="66.04" rot="R90"/>
 </instances>
 <busses>
@@
 <segment>
 <pinref part="S1" gate="1" pin="P"/>
-<wire x1="134.62" y1="93.98" x2="137.16" y2="93.98" width="0.1524" layer="91"/>
+<wire x1="99.06" y1="66.04" x2="101.6" y2="66.04" width="0.1524" layer="91"/>
 <pinref part="SUPPLY1" gate="GND" pin="GND"/>
 </segment>
@@
 <wire x1="190.5" y1="142.24" x2="193.04" y2="142.24" width="0.1524" layer="91"/>
 <label x="187.96" y="142.24" size="1.778" layer="95"/>
-</segment>
-</net>
-<net name="D1" class="0">
-<segment>
-<pinref part="U$1" gate="G$1" pin="RX1"/>
-<wire x1="111.76" y1="96.52" x2="116.84" y2="96.52" width="0.1524" layer="91"/>
-<label x="116.84" y="96.52" size="1.27" layer="95" xref="yes"/>
-</segment>
-<segment>
-<pinref part="D1" gate="G$1" pin="A"/>
-<wire x1="190.5" y1="149.86" x2="193.04" y2="149.86" width="0.1524" layer="91"/>
-<label x="187.96" y="149.86" size="1.778" layer="95"/>
-</segment>
-</net>
-<net name="N$1" class="0">
-<segment>
-<pinref part="U$1" gate="G$1" pin="TX0"/>
-<pinref part="S1" gate="1" pin="S"/>
-<wire x1="111.76" y1="93.98" x2="124.46" y2="93.98" width="0.1524" layer="91"/>
 </segment>
 </net>
@@
 </segment>
 </net>
+<net name="A1" class="0">
+<segment>
+<pinref part="U$1" gate="G$1" pin="A1"/>
+<wire x1="78.74" y1="119.38" x2="76.2" y2="119.38" width="0.1524" layer="91"/>
+<label x="76.2" y="119.38" size="1.27" layer="95" rot="R180" xref="yes"/>
+</segment>
+<segment>
+<pinref part="D1" gate="G$1" pin="A"/>
+<wire x1="190.5" y1="149.86" x2="193.04" y2="149.86" width="0.1524" layer="91"/>
+<label x="187.96" y="149.86" size="1.778" layer="95"/>
+</segment>
+</net>
+<net name="A3" class="0">
+<segment>
+<pinref part="U$1" gate="G$1" pin="A3"/>
+<wire x1="78.74" y1="114.3" x2="76.2" y2="114.3" width="0.1524" layer="91"/>
+<label x="76.2" y="114.3" size="1.27" layer="95" rot="R180" xref="yes"/>
+</segment>
+<segment>
+<pinref part="S1" gate="1" pin="S"/>
+<wire x1="88.9" y1="66.04" x2="83.82" y2="66.04" width="0.1524" layer="91"/>
+<label x="78.74" y="66.04" size="1.778" layer="95"/>
+</segment>
+</net>
